File: kicad/DoorSensor/DoorSensor.kicad_sch (KiCad schematic)
At the start: 7 parts, among them J1 AVR-ISP-6, J3 ADXL345 Module, U1 ATtiny44A-P, U2 NRF24L01_Breakout

Commit message: simavr support; initial board layout
Parts:
- BT1: footprint (none) -> TerminalBlock_4Ucon:TerminalBlock_4Ucon_1x02_P3.50mm_Horizontal
- C1: value C -> 0.1u; footprint (none) -> Capacitor_THT:C_Disc_D4.3mm_W1.9mm_P5.00mm
- C2: value C_Small -> 0.1u; footprint (none) -> Capacitor_THT:C_Disc_D4.3mm_W1.9mm_P5.00mm
- J1: footprint (none) -> Connector_IDC:IDC-Header_2x03_P2.54mm_Vertical
- J3: footprint (none) -> Connector_PinHeader_2.54mm:PinHeader_1x08_P2.54mm_Vertical
Connections:
- net +BATT: now also C2.2; no longer J1.2 (VCC)
- net GND: no longer C2.2
- net SCL: now also U1.3 (XTAL2/PB1)
- net SDA: now also U1.2 (XTAL1/PB0)
- net ACCEL_INT1: now reaches U1.5 (PB2)
- net ACCEL_INT1: now also J3.4 (Pin_4)
- net NRF_IRQ: now reaches U1.6 (PA7)
- net NRF_IRQ: now also U2.8 (IRQ)
- net ACCEL_SELECT: no longer names the net of U1.12 (PA1)
- net ACCEL_SELECT: no longer J3.3 (Pin_3)
- no-connect marks 4 -> 7
Other:
- moved on the sheet: BT1, C1, C2, J1, J3, U1, U2
